File: PCB/usb.kicad_sch (KiCad schematic)
At the start: 0 parts

Commit message: Add power supplies
Parts:
- added J1: 918-418K2023S40001, Connector_USB:USB_C_Receptacle_GCT_USB4105-xx-A_16P_TopMnt_Horizontal, symbol Connector:USB_C_Receptacle_USB2.0_16P
- added R1, R2: 5.1kΩ, Resistor_SMD:R_0402_1005Metric_Pad0.72x0.64mm_HandSolder, symbol Device:R
Connections:
- new net: J1.A5 (CC1), R2.1
- new net: J1.A6 (D+), J1.B6 (D+)
- new net: J1.A7 (D-), J1.B7 (D-)
- new net: J1.B5 (CC2), R1.1
- new net GND: J1.A1 (GND), J1.A12 (GND), J1.B1 (GND), J1.B12 (GND), J1.S1 (SHIELD), R1.2, R2.2
- new net VBUS: J1.A4 (VBUS), J1.A9 (VBUS), J1.B4 (VBUS), J1.B9 (VBUS)
- no-connect marks 0 -> 2
