File: PCB/clavier.kicad_pcb (KiCad board)
At the start: 4 copper layers, 434 x 134 mm, 141 parts, among them J1 TC2050, SW1 Esc, SW10 F9, SW100 Steuerung, SW101 ←, SW102 ↓, SW103 →, SW104 0, SW105 Komma, SW106 Eingabe, SW11 F10, SW12 F11, SW13 F12, SW14 Druck, SW15 Rollen, SW16 Pause, SW17 Sperren, SW18 Zirkumflex, SW19 1, SW2 F1, SW20 2, SW21 3, SW22 4, SW23 5, SW24 6, SW25 7, SW26 8, SW27 9, SW28 0, SW29 Eszett, SW3 F2, SW30 Akut, SW31 Rücktaste, SW32 Einfügen, SW33 Pos1, SW34 Bild↑, SW35 NumLock, SW36 Schrägstrich, SW37 Sternchen, SW38 Minus, SW39 Tab, SW4 F3, SW40 Q, SW41 W, SW42 E, SW43 R, SW44 T, SW45 Z, SW46 U, SW47 I, SW48 O, SW49 P, SW5 F4, SW50 Ü, SW51 Plus, SW52 Eingabe, SW53 Entfernen, SW54 Ende, SW55 Bild↓, SW56 7, SW57 8, SW58 9, SW59 Compose, SW6 F5, SW60 A, SW61 S, SW62 D, SW63 F, SW64 G, SW65 H, SW66 J, SW67 K, SW68 L, SW69 Ö, SW7 F6, SW70 Ä, SW71 Raute, SW72 4, SW73 5, SW74 6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

Commit message: Add more TODOs
Parts:
- moved C13 611.1 mm to (-172.2, -26.4)
- moved Y1 611.1 mm to (-172.2, -23.4)
- moved U1 19.0 mm to (382.5, 210.6)
- moved SW5 10.6 mm to (199.8, 138.9)
- moved SW1 4.62 mm to (95.3, 138.9)
- moved SW10 4.62 mm to (304.3, 138.9)
- moved SW11 4.62 mm to (323.3, 138.9)
- moved SW12 4.62 mm to (342.3, 138.9)
- moved SW13 4.62 mm to (361.3, 138.9)
- moved SW14 4.62 mm to (385.0, 138.9)
- moved SW15 4.62 mm to (404.0, 138.9)
- moved SW16 4.62 mm to (423.0, 138.9)
- moved SW17 4.62 mm to (503.8, 138.9)
- moved SW2 4.62 mm to (133.3, 138.9)
- moved SW3 4.62 mm to (152.3, 138.9)
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Routing:
- added copper zone on B.Cu, net GND
- added copper zone on F.Cu, net GND

Commit message: Add power supplies
Parts:
- added C27: 10µF, Capacitor_SMD:C_0805_2012Metric, F.Cu at (53.6, 57.1)
- added C28: 22µF, Capacitor_SMD:C_0805_2012Metric, F.Cu at (53.6, 63.1)
- added C29: 22µF, Capacitor_SMD:C_0805_2012Metric, F.Cu at (58.1, 57.1)
- added C30: 10µF, Capacitor_SMD:C_0805_2012Metric, F.Cu at (53.6, 60.1)
- added C31: 22µF, Capacitor_SMD:C_0805_2012Metric, F.Cu at (58.1, 60.1)
- added C32: 22µF, Capacitor_SMD:C_0805_2012Metric, F.Cu at (58.1, 63.1)
- added C33: 10µF, Capacitor_SMD:C_0805_2012Metric, F.Cu at (62.5, 57.1)
- added C34: 22µF, Capacitor_SMD:C_0805_2012Metric, F.Cu at (62.5, 60.1)
- added C35: 22µF, Capacitor_SMD:C_0805_2012Metric, F.Cu at (62.5, 63.1)
- added J1: 918-418K2023S40001, Connector_USB:USB_C_Receptacle_GCT_USB4105-xx-A_16P_TopMnt_Horizontal, F.Cu at (73.3, 60.9)
- added L1: 2.2µH, Inductor_SMD:L_1210_3225Metric, F.Cu at (54.2, 66.7)
- added L2: 2.2µH, Inductor_SMD:L_1210_3225Metric, F.Cu at (54.2, 71.0)
- added L3: 2.2µH, Inductor_SMD:L_1210_3225Metric, F.Cu at (54.2, 75.2)
- added R1: 5.1kΩ, Resistor_SMD:R_0402_1005Metric_Pad0.72x0.64mm_HandSolder, F.Cu at (69.1, 66.6)
- added R10: 4.75kΩ, Resistor_SMD:R_0402_1005Metric_Pad0.72x0.64mm_HandSolder, F.Cu at (63.8, 71.6)
- added R11: 1.5kΩ, Resistor_SMD:R_0402_1005Metric_Pad0.72x0.64mm_HandSolder, F.Cu at (63.8, 69.6)
- added R12: 1.37kΩ, Resistor_SMD:R_0402_1005Metric_Pad0.72x0.64mm_HandSolder, F.Cu at (63.8, 75.6)
- added R13: 1.65kΩ, Resistor_SMD:R_0402_1005Metric_Pad0.72x0.64mm_HandSolder, F.Cu at (63.8, 73.6)
- added R2: 5.1kΩ, Resistor_SMD:R_0402_1005Metric_Pad0.72x0.64mm_HandSolder, F.Cu at (69.1, 68.6)
- added R8: 11.5kΩ, Resistor_SMD:R_0402_1005Metric_Pad0.72x0.64mm_HandSolder, F.Cu at (63.8, 67.6)
- added R9: 2.55kΩ, Resistor_SMD:R_0402_1005Metric_Pad0.72x0.64mm_HandSolder, F.Cu at (63.8, 65.6)
- added U3: TLV62569DBVR, Package_TO_SOT_SMD:SOT-23-5, F.Cu at (59.6, 67.0)
- added U4: TLV62569DBVR, Package_TO_SOT_SMD:SOT-23-5, F.Cu at (59.6, 71.7)
- added U5: TLV62569DBVR, Package_TO_SOT_SMD:SOT-23-5, F.Cu at (59.6, 76.3)
- C1, C10, C11, C12, C13, C2, C3, C4, C5, C6, C7, C8, C9: footprint Capacitor_SMD:C_0603_1608Metric -> Capacitor_SMD:C_0402_1005Metric_Pad0.74x0.62mm_HandSolder
- C14: renamed from C24; footprint Capacitor_SMD:C_0603_1608Metric -> Capacitor_SMD:C_0402_1005Metric_Pad0.74x0.62mm_HandSolder
- C15: renamed from C25; footprint Capacitor_SMD:C_0603_1608Metric -> Capacitor_SMD:C_0402_1005Metric_Pad0.74x0.62mm_HandSolder
- C16: renamed from C26; footprint Capacitor_SMD:C_0603_1608Metric -> Capacitor_SMD:C_0402_1005Metric_Pad0.74x0.62mm_HandSolder
- C17: renamed from C14; footprint Capacitor_SMD:C_0603_1608Metric -> Capacitor_SMD:C_0402_1005Metric_Pad0.74x0.62mm_HandSolder
- C18: renamed from C15; footprint Capacitor_SMD:C_0603_1608Metric -> Capacitor_SMD:C_0402_1005Metric_Pad0.74x0.62mm_HandSolder
- C19: renamed from C16; footprint Capacitor_SMD:C_0603_1608Metric -> Capacitor_SMD:C_0402_1005Metric_Pad0.74x0.62mm_HandSolder
- C20: renamed from C17; footprint Capacitor_SMD:C_0603_1608Metric -> Capacitor_SMD:C_0402_1005Metric_Pad0.74x0.62mm_HandSolder
- C21: renamed from C18; footprint Capacitor_SMD:C_0603_1608Metric -> Capacitor_SMD:C_0402_1005Metric_Pad0.74x0.62mm_HandSolder
- C22: renamed from C19; footprint Capacitor_SMD:C_0603_1608Metric -> Capacitor_SMD:C_0402_1005Metric_Pad0.74x0.62mm_HandSolder
- C23: renamed from C20; footprint Capacitor_SMD:C_0603_1608Metric -> Capacitor_SMD:C_0402_1005Metric_Pad0.74x0.62mm_HandSolder
- C24: renamed from C21; footprint Capacitor_SMD:C_0603_1608Metric -> Capacitor_SMD:C_0402_1005Metric_Pad0.74x0.62mm_HandSolder
- C25: renamed from C22; footprint Capacitor_SMD:C_0603_1608Metric -> Capacitor_SMD:C_0402_1005Metric_Pad0.74x0.62mm_HandSolder
- C26: renamed from C23; footprint Capacitor_SMD:C_0603_1608Metric -> Capacitor_SMD:C_0402_1005Metric_Pad0.74x0.62mm_HandSolder
- R3: renamed from R1; value 10k -> 10kΩ; footprint Resistor_SMD:R_0603_1608Metric -> Resistor_SMD:R_0402_1005Metric_Pad0.72x0.64mm_HandSolder
- R4: renamed from R2; value 10k -> 10kΩ; footprint Resistor_SMD:R_0603_1608Metric -> Resistor_SMD:R_0402_1005Metric_Pad0.72x0.64mm_HandSolder
- R5: renamed from R3; value 10k -> 10kΩ; footprint Resistor_SMD:R_0603_1608Metric -> Resistor_SMD:R_0402_1005Metric_Pad0.72x0.64mm_HandSolder
- R6: renamed from R4; value 10k -> 10kΩ; footprint Resistor_SMD:R_0603_1608Metric -> Resistor_SMD:R_0402_1005Metric_Pad0.72x0.64mm_HandSolder
- R7: renamed from R5; value 1k -> 1kΩ; footprint Resistor_SMD:R_0603_1608Metric -> Resistor_SMD:R_0402_1005Metric_Pad0.72x0.64mm_HandSolder
- SW1: value Esc -> ~
- SW10: value F9 -> ~
- SW100, SW93: value Steuerung -> ~
- SW101: value ← -> ~
- SW102: value ↓ -> ~
- SW103: value → -> ~
- SW104, SW28: value 0 -> ~
- SW105, SW85: value Komma -> ~
- SW106, SW52: value Eingabe -> ~
- SW11: value F10 -> ~
- SW12: value F11 -> ~
- SW13: value F12 -> ~
- SW14: value Druck -> ~
- SW15: value Rollen -> ~
- SW16: value Pause -> ~
- SW17: value Sperren -> ~
- SW18: value Zirkumflex -> ~
- SW19, SW90: value 1 -> ~
- SW2: value F1 -> ~
- SW20, SW91: value 2 -> ~
- SW21, SW92: value 3 -> ~
- SW22, SW72: value 4 -> ~
- SW23, SW73: value 5 -> ~
- SW24, SW74: value 6 -> ~
- SW25, SW56: value 7 -> ~
- SW26, SW57: value 8 -> ~
- SW27, SW58: value 9 -> ~
- SW29: value Eszett -> ~
- SW3: value F2 -> ~
- SW30: value Akut -> ~
- SW31: value Rücktaste -> ~
- SW32: value Einfügen -> ~
- SW33: value Pos1 -> ~
- SW34: value Bild↑ -> ~
- SW35: value NumLock -> ~
- SW36: value Schrägstrich -> ~
- SW37: value Sternchen -> ~
- SW38, SW87: value Minus -> ~
- SW39: value Tab -> ~
- SW4: value F3 -> ~
- SW40: value Q -> ~
- SW41: value W -> ~
- SW42: value E -> ~
- SW43: value R -> ~
- SW44: value T -> ~
- SW45: value Z -> ~
- SW46: value U -> ~
- SW47: value I -> ~
- SW48: value O -> ~
- SW49: value P -> ~
- SW5: value F4 -> ~
- SW50: value Ü -> ~
- SW51, SW75: value Plus -> ~
- SW53: value Entfernen -> ~
- SW54: value Ende -> ~
- SW55: value Bild↓ -> ~
- SW59: value Compose -> ~
- SW6: value F5 -> ~
- SW60: value A -> ~
- SW61: value S -> ~
- SW62: value D -> ~
- SW63: value F -> ~
- SW64: value G -> ~
- SW65: value H -> ~
- SW66: value J -> ~
- SW67: value K -> ~
- SW68: value L -> ~
- SW69: value Ö -> ~
- SW7: value F6 -> ~
- SW70: value Ä -> ~
- SW71: value Raute -> ~
- SW76, SW88: value Umschalt -> ~
- SW77: value < -> ~
- SW78: value Y -> ~
- SW79: value X -> ~
- SW8: value F7 -> ~
- SW80: value C -> ~
- SW81: value V -> ~
- SW82: value B -> ~
- SW83: value N -> ~
- SW84: value M -> ~
- SW86: value Punkt -> ~
- SW89: value ↑ -> ~
- SW9: value F8 -> ~
- SW94, SW98: value Meta -> ~
- SW95: value Alt -> ~
- SW96: value Leertaste -> ~
- SW97: value AltGr -> ~
- SW99: value Menü -> ~
- U1: value LFE5U-25F-6BG256x -> LFE5U-25F-6BG256C
- U2: value W25Q128JVS -> W25Q128JVSIQ
- Y1: value KC2520Z -> CO22H4-48.000-WPJDTSTL
- moved C1 283.9 mm to (104.1, 71.0)
- moved C10 283.9 mm to (112.1, 73.5)
- moved C11 283.9 mm to (112.1, 76.0)
- moved C12 283.9 mm to (112.1, 78.5)
- moved C13 283.9 mm to (87.2, 88.9)
- moved C14 283.9 mm to (75.5, 71.0)
- moved C15 283.9 mm to (75.5, 73.5)
- moved C16 283.9 mm to (75.5, 76.0)
- moved C17 283.9 mm to (94.1, 71.0)
- moved C18 283.9 mm to (94.1, 73.5)
- moved C19 283.9 mm to (94.1, 76.0)
- moved C2 283.9 mm to (104.1, 73.5)
- moved C20 283.9 mm to (94.1, 78.5)
- moved C21 283.9 mm to (94.1, 81.0)
- moved C22 283.9 mm to (98.1, 71.0)
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- renumbered J1 to J2
Connections:
- net /Keys/K.A renamed /FPGA/K.A
- net /Keys/K.AE renamed /FPGA/K.AE
- net /Keys/K.Acute renamed /FPGA/K.Acute
- net /Keys/K.Alt renamed /FPGA/K.Alt
- net /Keys/K.AltGr renamed /FPGA/K.AltGr
- net /Keys/K.B renamed /FPGA/K.B
- net /Keys/K.Bksp renamed /FPGA/K.Bksp
- net /Keys/K.C renamed /FPGA/K.C
- net /Keys/K.Circ renamed /FPGA/K.Circ
- net /Keys/K.Comma renamed /FPGA/K.Comma
- net /Keys/K.Comp renamed /FPGA/K.Comp
- net /Keys/K.D renamed /FPGA/K.D
- net /Keys/K.Delete renamed /FPGA/K.Delete
- net /Keys/K.Dot renamed /FPGA/K.Dot
- net /Keys/K.Down renamed /FPGA/K.Down
- net /Keys/K.E renamed /FPGA/K.E
- net /Keys/K.End renamed /FPGA/K.End
- net /Keys/K.Eszett renamed /FPGA/K.Eszett
- net /Keys/K.F renamed /FPGA/K.F
- net /Keys/K.G renamed /FPGA/K.G
- net /Keys/K.H renamed /FPGA/K.H
- net /Keys/K.Hash renamed /FPGA/K.Hash
- net /Keys/K.Home renamed /FPGA/K.Home
- net /Keys/K.I renamed /FPGA/K.I
- net /Keys/K.Insert renamed /FPGA/K.Insert
- net /Keys/K.J renamed /FPGA/K.J
- net /Keys/K.K renamed /FPGA/K.K
- net /Keys/K.L renamed /FPGA/K.L
- net /Keys/K.LCtrl renamed /FPGA/K.LCtrl
- net /Keys/K.LMeta renamed /FPGA/K.LMeta
- net /Keys/K.LShift renamed /FPGA/K.LShift
- net /Keys/K.Left renamed /FPGA/K.Left
- net /Keys/K.Lt renamed /FPGA/K.Lt
- net /Keys/K.M renamed /FPGA/K.M
- net /Keys/K.Menu renamed /FPGA/K.Menu
- net /Keys/K.Minus renamed /FPGA/K.Minus
- net /Keys/K.N renamed /FPGA/K.N
- net /Keys/K.O renamed /FPGA/K.O
- net /Keys/K.OE renamed /FPGA/K.OE
- net /Keys/K.P renamed /FPGA/K.P
- net /Keys/K.PgDn renamed /FPGA/K.PgDn
- net /Keys/K.PgUp renamed /FPGA/K.PgUp
- net /Keys/K.Plus renamed /FPGA/K.Plus
- net /Keys/K.Print renamed /FPGA/K.Print
- net /Keys/K.Q renamed /FPGA/K.Q
- net /Keys/K.R renamed /FPGA/K.R
- net /Keys/K.RCtrl renamed /FPGA/K.RCtrl
- net /Keys/K.RMeta renamed /FPGA/K.RMeta
- net /Keys/K.RShift renamed /FPGA/K.RShift
- net /Keys/K.Right renamed /FPGA/K.Right
- net /Keys/K.Rtrn renamed /FPGA/K.Rtrn
- net /Keys/K.S renamed /FPGA/K.S
- net /Keys/K.SLock renamed /FPGA/K.SLock
- net /Keys/K.Space renamed /FPGA/K.Space
- net /Keys/K.T renamed /FPGA/K.T
- net /Keys/K.Tab renamed /FPGA/K.Tab
- net /Keys/K.U renamed /FPGA/K.U
- net /Keys/K.UE renamed /FPGA/K.UE
- net /Keys/K.Up renamed /FPGA/K.Up
- net /Keys/K.V renamed /FPGA/K.V
- net /Keys/K.W renamed /FPGA/K.W
- net /Keys/K.X renamed /FPGA/K.X
- net /Keys/K.Y renamed /FPGA/K.Y
- net /Keys/K.Z renamed /FPGA/K.Z
- net /Keys/K._0 renamed /FPGA/K._0
- net /Keys/K._1 renamed /FPGA/K._1
- net /Keys/K._2 renamed /FPGA/K._2
- net /Keys/K._3 renamed /FPGA/K._3
- net /Keys/K._4 renamed /FPGA/K._4
- net /Keys/K._5 renamed /FPGA/K._5
- net /Keys/K._6 renamed /FPGA/K._6
- net /Keys/K._7 renamed /FPGA/K._7
- net /Keys/K._8 renamed /FPGA/K._8
- net /Keys/K._9 renamed /FPGA/K._9
- net /Keys/Kp.Dot renamed /FPGA/Kp.Dot
- net /Keys/Kp.Minus renamed /FPGA/Kp.Minus
- net /Keys/Kp.NLock renamed /FPGA/Kp.NLock
- net /Keys/Kp.Plus renamed /FPGA/Kp.Plus
- net /Keys/Kp.Rtrn renamed /FPGA/Kp.Rtrn
- net /Keys/Kp.Slash renamed /FPGA/Kp.Slash
- net /Keys/Kp.Star renamed /FPGA/Kp.Star
- net /Keys/Kp._0 renamed /FPGA/Kp._0
- net /Keys/Kp._1 renamed /FPGA/Kp._1
- net /Keys/Kp._2 renamed /FPGA/Kp._2
- net /Keys/Kp._3 renamed /FPGA/Kp._3
- net /Keys/Kp._4 renamed /FPGA/Kp._4
- net /Keys/Kp._5 renamed /FPGA/Kp._5
- net /Keys/Kp._6 renamed /FPGA/Kp._6
- net /Keys/Kp._7 renamed /FPGA/Kp._7
- net /Keys/Kp._8 renamed /FPGA/Kp._8
- net /Keys/Kp._9 renamed /FPGA/Kp._9

Commit message: Add a USB hub
Parts:
- added C1: 1µF, Capacitor_SMD:C_0402_1005Metric_Pad0.74x0.62mm_HandSolder, F.Cu at (145.8, 55.2)
- added C2: 100nF, Capacitor_SMD:C_0402_1005Metric_Pad0.74x0.62mm_HandSolder, F.Cu at (145.8, 57.2)
- added C3: 1µF, Capacitor_SMD:C_0402_1005Metric_Pad0.74x0.62mm_HandSolder, F.Cu at (145.8, 59.2)
- added C4: 100nF, Capacitor_SMD:C_0402_1005Metric_Pad0.74x0.62mm_HandSolder, F.Cu at (145.8, 61.1)
- added C5: 1µF, Capacitor_SMD:C_0402_1005Metric_Pad0.74x0.62mm_HandSolder, F.Cu at (145.8, 63.1)
- added C6: 1µF, Capacitor_SMD:C_0402_1005Metric_Pad0.74x0.62mm_HandSolder, F.Cu at (145.8, 65.1)
- added J2: 901-211A1021D10100, Connector_USB:USB_A_Molex_67643_Horizontal, F.Cu at (128.3, 57.5)
- added J3: 901-211A1021D10100, Connector_USB:USB_A_Molex_67643_Horizontal, F.Cu at (128.3, 74.8)
- added L1: 2.2µH, Inductor_SMD:L_1210_3225Metric, F.Cu at (143.7, 81.5)
- added R10: 100kΩ, Resistor_SMD:R_0402_1005Metric_Pad0.72x0.64mm_HandSolder, F.Cu at (142.6, 69.2)
- added R11: 680Ω, Resistor_SMD:R_0402_1005Metric_Pad0.72x0.64mm_HandSolder, F.Cu at (142.6, 71.2)
- added R3: 100kΩ, Resistor_SMD:R_0402_1005Metric_Pad0.72x0.64mm_HandSolder, F.Cu at (142.6, 55.2)
- added R4: 10kΩ, Resistor_SMD:R_0402_1005Metric_Pad0.72x0.64mm_HandSolder, F.Cu at (142.6, 57.2)
- added R5: 100kΩ, Resistor_SMD:R_0402_1005Metric_Pad0.72x0.64mm_HandSolder, F.Cu at (142.6, 59.2)
- added R6: 47kΩ, Resistor_SMD:R_0402_1005Metric_Pad0.72x0.64mm_HandSolder, F.Cu at (142.6, 61.2)
- added R7: 100kΩ, Resistor_SMD:R_0402_1005Metric_Pad0.72x0.64mm_HandSolder, F.Cu at (142.6, 63.2)
- added R8: 100kΩ, Resistor_SMD:R_0402_1005Metric_Pad0.72x0.64mm_HandSolder, F.Cu at (142.6, 65.2)
- added R9: 100kΩ, Resistor_SMD:R_0402_1005Metric_Pad0.72x0.64mm_HandSolder, F.Cu at (142.6, 67.2)
- added U1: GL852G-OHY60, Package_DFN_QFN:QFN-28-1EP_5x5mm_P0.5mm_EP3.75x3.75mm, F.Cu at (144.6, 75.8)
- added Y1: CO22H4-12.000-WPGDTSNL, Oscillator:Oscillator_SMD_Kyocera_KC2520Z-4Pin_2.5x2.0mm, F.Cu at (142.9, 85.9)
- added Y2: CO22H4-12.000-WPGDTSNL, Oscillator:Oscillator_SMD_Kyocera_KC2520Z-4Pin_2.5x2.0mm, F.Cu at (152.2, 56.5)
- renumbered C4 to C10, C5 to C11, C6 to C12, C7 to C13, C8 to C14, C9 to C15, C10 to C16, C11 to C17, C12 to C18, C13 to C19, C14 to C20, C15 to C21, C16 to C22, C17 to C23, C18 to C24, C19 to C25, C20 to C26, C21 to C27, C22 to C28, C23 to C29, C24 to C30, C25 to C31, C26 to C32, C27 to C33, C28 to C34, C29 to C35, C30 to C36, C31 to C37, C32 to C38, C33 to C39, C34 to C40, C35 to C41, C1 to C7, C2 to C8, C3 to C9, J2 to J4, L1 to L2, L2 to L3, L3 to L4, R3 to R12, R4 to R13, R5 to R14, R6 to R15, R7 to R16, R8 to R17, R9 to R18, R10 to R19, R11 to R20, R12 to R21, R13 to R22, U1 to U2, U2 to U3, U3 to U4, U4 to U5, U5 to U6
Connections:
- net Net-(J1-D+-PadA6) renamed /USB hub/D+
- net Net-(J1-D--PadA7) renamed /USB hub/D-
- U2 pad A10: unconnected-(U1C-PT42B-PadA10) -> /FPGA/K.T
- U2 pad A11: unconnected-(U1C-PT53A-PadA11) -> /FPGA/K.F3
- U2 pad A12: unconnected-(U1C-PT53B-PadA12) -> /FPGA/K.Lt
- U2 pad A13: unconnected-(U1C-PT65A-PadA13) -> /FPGA/Kp._7
- U2 pad A14: unconnected-(U1C-PT65B-PadA14) -> /FPGA/Kp.Minus
- U2 pad A15: unconnected-(U1C-PT67B-PadA15) -> /FPGA/K.AltGr
- U2 pad A2: /FPGA/K.Esc -> /FPGA/FPGA_IO0
- U2 pad A3: /FPGA/K.F1 -> /FPGA/Kp._6
- U2 pad A4: /FPGA/K.F2 -> /FPGA/FPGA_IO3
- U2 pad A5: /FPGA/K.F9 -> /FPGA/K.Dot
- U2 pad A6: /FPGA/K.F10 -> /FPGA/K.AE
- U2 pad A7: unconnected-(U1B-PT29A-PadA7) -> /FPGA/USB_FPGA-
- U2 pad A8: unconnected-(U1B-PT29B-PadA8) -> /FPGA/USB_FPGA+
- U2 pad A9: unconnected-(U1C-PT42A-PadA9) -> /FPGA/Kp._5
- U2 pad B1: unconnected-(U1G-PL2A-PadB1) -> /FPGA/FPGA_IO152
- U2 pad B10: unconnected-(U1C-PT44A-PadB10) -> /FPGA/FPGA_IO34
- U2 pad B11: unconnected-(U1C-PT49A-PadB11) -> /FPGA/K.F2
- U2 pad B12: unconnected-(U1C-PT56A-PadB12) -> /FPGA/K.PgDn
- U2 pad B13: unconnected-(U1C-PT60A-PadB13) -> /FPGA/K.LCtrl
- U2 pad B14: unconnected-(U1C-PT67A-PadB14) -> /FPGA/K.W
- U2 pad B15: unconnected-(U1D-PR2B-PadB15) -> /FPGA/FPGA_IO57
- U2 pad B16: unconnected-(U1D-PR2A-PadB16) -> /FPGA/FPGA_IO56
- U2 pad B2: unconnected-(U1G-PL2B-PadB2) -> /FPGA/K.SLock
- U2 pad B3: unconnected-(U1B-PT4B-PadB3) -> /FPGA/K.Down
- U2 pad B4: /FPGA/K.F5 -> /FPGA/K.Delete
- U2 pad B5: unconnected-(U1B-PT15B-PadB5) -> /FPGA/FPGA_IO11
- U2 pad B6: unconnected-(U1B-PT22B-PadB6) -> /FPGA/K.D
- U2 pad B7: unconnected-(U1B-PT27B-PadB7) -> /FPGA/K.Menu
- U2 pad B8: unconnected-(U1C-PT35B-PadB8) -> /FPGA/K.F9
- U2 pad B9: unconnected-(U1C-PT38A-PadB9) -> /FPGA/FPGA_IO28
- U2 pad C1: unconnected-(U1G-PL5A-PadC1) -> /FPGA/FPGA_IO156
- U2 pad C10: unconnected-(U1C-PT44B-PadC10) -> /FPGA/K.F7
- U2 pad C11: unconnected-(U1C-PT49B-PadC11) -> /FPGA/K.I
- U2 pad C12: unconnected-(U1C-PT56B-PadC12) -> /FPGA/K.Esc
- U2 pad C13: unconnected-(U1C-PT60B-PadC13) -> /FPGA/K.Tab
- U2 pad C14: unconnected-(U1D-PR2C-PadC14) -> /FPGA/K.H
- U2 pad C15: unconnected-(U1D-PR5B-PadC15) -> /FPGA/FPGA_IO61
- U2 pad C16: unconnected-(U1D-PR5A-PadC16) -> /FPGA/K.End
- U2 pad C2: unconnected-(U1G-PL5B-PadC2) -> /FPGA/K.PgUp
- U2 pad C3: unconnected-(U1G-PL2C-PadC3) -> /FPGA/K.Space
- U2 pad C4: unconnected-(U1B-PT11A-PadC4) -> /FPGA/FPGA_IO6
- U2 pad C5: /FPGA/K.F8 -> /FPGA/K.L
- U2 pad C6: unconnected-(U1B-PT22A-PadC6) -> /FPGA/FPGA_IO16
- U2 pad C7: unconnected-(U1B-PT27A-PadC7) -> /FPGA/Kp._1
- U2 pad C8: unconnected-(U1C-PT35A-PadC8) -> /FPGA/FPGA_IO26
- U2 pad C9: unconnected-(U1C-PT38B-PadC9) -> /FPGA/K._8
- U2 pad D1: unconnected-(U1G-PL8A-PadD1) -> /FPGA/FPGA_IO160
- U2 pad D10: unconnected-(U1C-PT47A-PadD10) -> /FPGA/K.Rtrn
- U2 pad D11: unconnected-(U1C-PT51A-PadD11) -> /FPGA/K._6
- U2 pad D12: unconnected-(U1C-PT58A-PadD12) -> /FPGA/FPGA_IO46
- U2 pad D13: unconnected-(U1C-PT62A-PadD13) -> /FPGA/K.R
- U2 pad D14: unconnected-(U1D-PR2D-PadD14) -> /FPGA/FPGA_IO59
- U2 pad D16: unconnected-(U1D-PR8A-PadD16) -> /FPGA/FPGA_IO64
- U2 pad D3: unconnected-(U1G-PL2D-PadD3) -> /FPGA/K.S
- U2 pad D4: /FPGA/K.F4 -> /FPGA/K.Eszett
- U2 pad D5: /FPGA/K.F7 -> /FPGA/K.F10
- U2 pad D6: /FPGA/K.F12 -> /FPGA/FPGA_IO15
- U2 pad D7: unconnected-(U1B-PT24B-PadD7) -> /FPGA/K.F4
- U2 pad D8: unconnected-(U1C-PT33B-PadD8) -> /FPGA/FPGA_IO25
- U2 pad D9: unconnected-(U1C-PT40A-PadD9) -> /FPGA/K.F8
- U2 pad E1: unconnected-(U1G-PL11D-PadE1) -> /FPGA/K.O
- U2 pad E10: unconnected-(U1C-PT47B-PadE10) -> /FPGA/K.F11
- U2 pad E11: unconnected-(U1C-PT51B-PadE11) -> /FPGA/K.Left
- U2 pad E12: unconnected-(U1C-PT58B-PadE12) -> /FPGA/K.Comma
- U2 pad E13: unconnected-(U1C-PT62B-PadE13) -> /FPGA/FPGA_IO51
- U2 pad E14: unconnected-(U1D-PR5C-PadE14) -> /FPGA/FPGA_IO62
- U2 pad E15: unconnected-(U1D-PR8B-PadE15) -> /FPGA/K.V
- U2 pad E16: unconnected-(U1D-PR11D-PadE16) -> /FPGA/FPGA_IO71
- U2 pad E2: unconnected-(U1G-PL8B-PadE2) -> /FPGA/K.A
- U2 pad E3: unconnected-(U1G-PL5C-PadE3) -> /FPGA/FPGA_IO158
- U2 pad E4: /FPGA/K.F3 -> /FPGA/K.Print
- U2 pad E5: /FPGA/K.F6 -> /FPGA/FPGA_IO8
- U2 pad E6: /FPGA/K.F11 -> /FPGA/FPGA_IO14
- U2 pad E7: unconnected-(U1B-PT24A-PadE7) -> /FPGA/K.Up
- U2 pad E8: unconnected-(U1C-PT33A-PadE8) -> /FPGA/Kp.Rtrn
- U2 pad E9: unconnected-(U1C-PT40B-PadE9) -> /FPGA/FPGA_IO31
- U2 pad F1: unconnected-(U1G-PL14A-PadF1) -> /FPGA/FPGA_IO168
- U2 pad F12: unconnected-(U1D-PR8D-PadF12) -> /FPGA/K.Comp
- U2 pad F13: unconnected-(U1D-PR8C-PadF13) -> /FPGA/K.Home
- U2 pad F14: unconnected-(U1D-PR5D-PadF14) -> /FPGA/FPGA_IO63
- U2 pad F15: unconnected-(U1D-PR11C-PadF15) -> /FPGA/K.Alt
- U2 pad F16: unconnected-(U1D-PR14A-PadF16) -> /FPGA/K._7
- U2 pad F2: unconnected-(U1G-PL11C-PadF2) -> /FPGA/FPGA_IO166
- U2 pad F3: unconnected-(U1G-PL5D-PadF3) -> /FPGA/FPGA_IO159
- U2 pad F4: unconnected-(U1G-PL8C-PadF4) -> /FPGA/K.OE
- U2 pad F5: unconnected-(U1G-PL8D-PadF5) -> /FPGA/FPGA_IO163
- U2 pad G1: unconnected-(U1G-PL20A-PadG1) -> /FPGA/FPGA_IO176
- U2 pad G12: unconnected-(U1D-PR11A-PadG12) -> /FPGA/K.Acute
- U2 pad G13: unconnected-(U1D-PR11B-PadG13) -> /FPGA/K.Pause
- U2 pad G14: unconnected-(U1D-PR14C-PadG14) -> /FPGA/K._9
- U2 pad G15: unconnected-(U1D-PR14B-PadG15) -> /FPGA/FPGA_IO73
- U2 pad G16: unconnected-(U1D-PR20A-PadG16) -> /FPGA/Kp._9
- U2 pad G2: unconnected-(U1G-PL14B-PadG2) -> /FPGA/K.X
- U2 pad G3: unconnected-(U1G-PL14C-PadG3) -> /FPGA/FPGA_IO170
- U2 pad G4: unconnected-(U1G-PL11B-PadG4) -> /FPGA/K.N
- U2 pad G5: unconnected-(U1G-PL11A-PadG5) -> /FPGA/K._3
- U2 pad H12: unconnected-(U1D-PR17A-PadH12) -> /FPGA/K.C
- U2 pad H13: unconnected-(U1D-PR17B-PadH13) -> /FPGA/Kp._2
- U2 pad H14: unconnected-(U1D-PR14D-PadH14) -> /FPGA/K.F6
- U2 pad H15: unconnected-(U1D-PR20B-PadH15) -> /FPGA/K.F
- U2 pad H2: unconnected-(U1G-PL20B-PadH2) -> /FPGA/K.UE
- U2 pad H3: unconnected-(U1G-PL14D-PadH3) -> /FPGA/K.U
- U2 pad H4: unconnected-(U1G-PL17B-PadH4) -> /FPGA/FPGA_IO173
- U2 pad H5: unconnected-(U1G-PL17A-PadH5) -> /FPGA/FPGA_IO172
- U2 pad J1: unconnected-(U1G-PL23A-PadJ1) -> /FPGA/FPGA_IO180
- U2 pad J12: unconnected-(U1D-PR17D-PadJ12) -> /FPGA/K.F12
- U2 pad J13: unconnected-(U1D-PR17C-PadJ13) -> /FPGA/K._4
- U2 pad J14: unconnected-(U1D-PR20C-PadJ14) -> /FPGA/K.Minus
- U2 pad J15: unconnected-(U1D-PR23B-PadJ15) -> /FPGA/FPGA_IO85
- U2 pad J16: unconnected-(U1D-PR23A-PadJ16) -> /FPGA/K.RMeta
- U2 pad J2: unconnected-(U1G-PL23B-PadJ2) -> /FPGA/FPGA_IO181
- U2 pad J3: unconnected-(U1G-PL20C-PadJ3) -> /FPGA/FPGA_IO178
- U2 pad J4: unconnected-(U1G-PL17C-PadJ4) -> /FPGA/FPGA_IO174
- U2 pad J5: unconnected-(U1G-PL17D-PadJ5) -> /FPGA/K.Circ
- U2 pad K1: unconnected-(U1G-PL23C-PadK1) -> /FPGA/Kp.Slash
- U2 pad K12: unconnected-(U1E-PR29B-PadK12) -> /FPGA/K.P
- U2 pad K13: unconnected-(U1E-PR29A-PadK13) -> /FPGA/K._5
- U2 pad K14: unconnected-(U1D-PR20D-PadK14) -> /FPGA/K._0
- U2 pad K15: unconnected-(U1D-PR23D-PadK15) -> /FPGA/FPGA_IO87
- U2 pad K16: unconnected-(U1D-PR23C-PadK16) -> /FPGA/K._1
- U2 pad K2: unconnected-(U1G-PL23D-PadK2) -> /FPGA/K.Lock
- U2 pad K3: unconnected-(U1G-PL20D-PadK3) -> /FPGA/FPGA_IO179
- U2 pad K4: unconnected-(U1F-PL29A-PadK4) -> /FPGA/K.E
- U2 pad K5: unconnected-(U1F-PL29B-PadK5) -> /FPGA/K.F5
- U2 pad L1: unconnected-(U1F-PL26A-PadL1) -> /FPGA/FPGA_IO120
- U2 pad L12: unconnected-(U1E-PR29D-PadL12) -> /FPGA/K.M
- U2 pad L13: unconnected-(U1E-PR29C-PadL13) -> /FPGA/FPGA_IO94
- U2 pad L14: unconnected-(U1E-PR32C-PadL14) -> /FPGA/K.Right
- U2 pad L15: unconnected-(U1E-PR26B-PadL15) -> /FPGA/FPGA_IO89
- U2 pad L16: unconnected-(U1E-PR26A-PadL16) -> /FPGA/Kp.NLock
- U2 pad L2: unconnected-(U1F-PL26B-PadL2) -> /FPGA/FPGA_IO121
- U2 pad L3: unconnected-(U1F-PL32C-PadL3) -> /FPGA/K.F1
- U2 pad L4: unconnected-(U1F-PL29C-PadL4) -> /FPGA/K.Q
- U2 pad L5: unconnected-(U1F-PL29D-PadL5) -> /FPGA/K.RCtrl
- U2 pad M1: /FPGA/CLK_48MHz -> /FPGA/CLK_12MHz
- U2 pad M11: unconnected-(U1E-PR47A-PadM11) -> /FPGA/K.Plus
- U2 pad M12: unconnected-(U1E-PR44C-PadM12) -> /FPGA/Kp._0
- U2 pad M13: unconnected-(U1E-PR35C-PadM13) -> /FPGA/K.LShift
- U2 pad M14: unconnected-(U1E-PR32D-PadM14) -> /FPGA/FPGA_IO99
- U2 pad M15: unconnected-(U1E-PR26D-PadM15) -> /FPGA/FPGA_IO91
- U2 pad M16: unconnected-(U1E-PR26C-PadM16) -> /FPGA/FPGA_IO90
- U2 pad M2: unconnected-(U1F-PL26D-PadM2) -> /FPGA/FPGA_IO123
- U2 pad M3: unconnected-(U1F-PL32D-PadM3) -> /FPGA/FPGA_IO131
- U2 pad M4: unconnected-(U1F-PL35C-PadM4) -> /FPGA/FPGA_IO134
- U2 pad M5: unconnected-(U1F-PL44C-PadM5) -> /FPGA/K.B
- U2 pad M6: unconnected-(U1F-PL47A-PadM6) -> /FPGA/K.Insert
- U2 pad N1: unconnected-(U1F-PL32A-PadN1) -> /FPGA/FPGA_IO128
- U2 pad N11: unconnected-(U1E-PR47B-PadN11) -> /FPGA/Kp._8
- U2 pad N12: unconnected-(U1E-PR44D-PadN12) -> /FPGA/FPGA_IO115
- U2 pad N13: unconnected-(U1E-PR38A-PadN13) -> /FPGA/FPGA_IO104
- U2 pad N14: unconnected-(U1E-PR35D-PadN14) -> /FPGA/K.Y
- U2 pad N16: unconnected-(U1E-PR32A-PadN16) -> /FPGA/FPGA_IO96
- U2 pad N3: unconnected-(U1F-PL35D-PadN3) -> /FPGA/FPGA_IO135
- U2 pad N4: unconnected-(U1F-PL38A-PadN4) -> /FPGA/Kp.Dot
- U2 pad N5: unconnected-(U1F-PL44D-PadN5) -> /FPGA/FPGA_IO147
- U2 pad N6: unconnected-(U1F-PL47B-PadN6) -> /FPGA/K._2
- U2 pad P1: unconnected-(U1F-PL35A-PadP1) -> /FPGA/FPGA_IO132
- U2 pad P11: unconnected-(U1E-PR47C-PadP11) -> /FPGA/FPGA_IO118
- U2 pad P12: unconnected-(U1E-PR47D-PadP12) -> /FPGA/FPGA_IO119
- U2 pad P13: unconnected-(U1E-PR41A-PadP13) -> /FPGA/FPGA_IO108
- U2 pad P14: unconnected-(U1E-PR38B-PadP14) -> /FPGA/FPGA_IO105
- U2 pad P15: unconnected-(U1E-PR32B-PadP15) -> /FPGA/K.LMeta
- U2 pad P16: unconnected-(U1E-PR35A-PadP16) -> /FPGA/Kp.Star
- U2 pad P2: unconnected-(U1F-PL32B-PadP2) -> /FPGA/FPGA_IO129
- U2 pad P3: unconnected-(U1F-PL38B-PadP3) -> /FPGA/K.RShift
- U2 pad P4: unconnected-(U1F-PL41A-PadP4) -> /FPGA/FPGA_IO140
- U2 pad P5: unconnected-(U1F-PL47D-PadP5) -> /FPGA/FPGA_IO151
- U2 pad P6: unconnected-(U1F-PL47C-PadP6) -> /FPGA/K.Z
- U2 pad R1: unconnected-(U1F-PL35B-PadR1) -> /FPGA/K.J
- U2 pad R12: unconnected-(U1E-PR44A-PadR12) -> /FPGA/Kp._4
- U2 pad R13: unconnected-(U1E-PR41C-PadR13) -> /FPGA/FPGA_IO110
- U2 pad R14: unconnected-(U1E-PR41B-PadR14) -> /FPGA/FPGA_IO109
- U2 pad R15: unconnected-(U1E-PR38C-PadR15) -> /FPGA/K.G
- U2 pad R16: unconnected-(U1E-PR35B-PadR16) -> /FPGA/K.K
- U2 pad R2: unconnected-(U1F-PL38C-PadR2) -> /FPGA/FPGA_IO138
- U2 pad R3: unconnected-(U1F-PL41B-PadR3) -> /FPGA/K.Bksp
- U2 pad R4: unconnected-(U1F-PL41C-PadR4) -> /FPGA/FPGA_IO142
- U2 pad R5: unconnected-(U1F-PL44A-PadR5) -> /FPGA/FPGA_IO144
- U2 pad T13: unconnected-(U1E-PR44B-PadT13) -> /FPGA/FPGA_IO113
- U2 pad T14: unconnected-(U1E-PR41D-PadT14) -> /FPGA/K.Hash
- U2 pad T15: unconnected-(U1E-PR38D-PadT15) -> /FPGA/FPGA_IO107
- U2 pad T2: unconnected-(U1F-PL38D-PadT2) -> /FPGA/FPGA_IO139
- U2 pad T3: unconnected-(U1F-PL41D-PadT3) -> /FPGA/Kp.Plus
- U2 pad T4: unconnected-(U1F-PL44B-PadT4) -> /FPGA/Kp._3

Commit message: Add the USB to JTAG bridge
Parts:
- added C10: 1µF, Capacitor_SMD:C_0402_1005Metric_Pad0.74x0.62mm_HandSolder, F.Cu at (181.6, 70.5)
- added C11: 1µF, Capacitor_SMD:C_0402_1005Metric_Pad0.74x0.62mm_HandSolder, F.Cu at (181.6, 72.5)
- added C7: 20pF, Capacitor_SMD:C_0402_1005Metric_Pad0.74x0.62mm_HandSolder, F.Cu at (181.6, 64.6)
- added C8: 1µF, Capacitor_SMD:C_0402_1005Metric_Pad0.74x0.62mm_HandSolder, F.Cu at (181.6, 66.5)
- added C9: 20pF, Capacitor_SMD:C_0402_1005Metric_Pad0.74x0.62mm_HandSolder, F.Cu at (181.6, 68.5)
- added D1: LED, LED_SMD:LED_0603_1608Metric_Pad1.05x0.95mm_HandSolder, F.Cu at (185.5, 75.6)
- added D2: LED, LED_SMD:LED_0603_1608Metric_Pad1.05x0.95mm_HandSolder, F.Cu at (196.8, 59.1)
- added D3: LED, LED_SMD:LED_0603_1608Metric_Pad1.05x0.95mm_HandSolder, F.Cu at (196.8, 61.7)
- added D4: LED, LED_SMD:LED_0603_1608Metric_Pad1.05x0.95mm_HandSolder, F.Cu at (196.8, 64.3)
- added D5: LED, LED_SMD:LED_0603_1608Metric_Pad1.05x0.95mm_HandSolder, F.Cu at (196.8, 66.9)
- added D6: LED, LED_SMD:LED_0603_1608Metric_Pad1.05x0.95mm_HandSolder, F.Cu at (196.8, 69.5)
- added J4: Pin header, 2x4, Connector_PinHeader_2.54mm:PinHeader_2x04_P2.54mm_Vertical_SMD, F.Cu at (446.5, 152.5)
- added J5: Pin header, 2x4, Connector_PinHeader_2.54mm:PinHeader_2x04_P2.54mm_Vertical_SMD, F.Cu at (466.5, 152.5)
- added R12: 10kΩ, Resistor_SMD:R_0402_1005Metric_Pad0.72x0.64mm_HandSolder, F.Cu at (184.9, 77.9)
- added R13: 2.55kΩ, Resistor_SMD:R_0402_1005Metric_Pad0.72x0.64mm_HandSolder, F.Cu at (184.9, 79.9)
- added R19: 2.55kΩ, Resistor_SMD:R_0402_1005Metric_Pad0.72x0.64mm_HandSolder, F.Cu at (200.7, 58.8)
- added R20: 2.55kΩ, Resistor_SMD:R_0402_1005Metric_Pad0.72x0.64mm_HandSolder, F.Cu at (200.7, 60.8)
- added R21: 2.55kΩ, Resistor_SMD:R_0402_1005Metric_Pad0.72x0.64mm_HandSolder, F.Cu at (200.7, 62.8)
- added R22: 2.55kΩ, Resistor_SMD:R_0402_1005Metric_Pad0.72x0.64mm_HandSolder, F.Cu at (200.7, 64.8)
- added R23: 2.55kΩ, Resistor_SMD:R_0402_1005Metric_Pad0.72x0.64mm_HandSolder, F.Cu at (200.7, 66.8)
- added SW1: DSIC01LS-P, Button_Switch_SMD:SW_DIP_SPSTx01_Slide_6.7x4.1mm_W8.61mm_P2.54mm_LowProfile, F.Cu at (186.3, 60.7)
- added U2: CH347F, Package_DFN_QFN:QFN-28-1EP_4x4mm_P0.4mm_EP2.4x2.4mm, F.Cu at (186.4, 66.7)
- added Y2: 8MHz, Crystal:Crystal_SMD_3225-4Pin_3.2x2.5mm, F.Cu at (185.9, 72.1)
- Y1: value CO22H4-12.000-WPGDTSNL -> 12MHz; footprint Oscillator:Oscillator_SMD_Kyocera_KC2520Z-4Pin_2.5x2.0mm -> Crystal:Crystal_SMD_2520-4Pin_2.5x2.0mm
- Y3: renamed from Y2; value CO22H4-12.000-WPGDTSNL -> 12MHz; footprint Oscillator:Oscillator_SMD_Kyocera_KC2520Z-4Pin_2.5x2.0mm -> Crystal:Crystal_SMD_2520-4Pin_2.5x2.0mm
- moved J1 417.6 mm to (485.0, 130.5), turned to 180 degrees
- moved J2 351.5 mm to (470.0, 140.0), turned to 180 degrees
- moved J3 328.2 mm to (450.0, 140.0), turned to 180 degrees
- renumbered C7 to C12, C8 to C13, C9 to C14, C10 to C15, C11 to C16, C12 to C17, C13 to C18, C14 to C19, C15 to C20, C16 to C21, C17 to C22, C18 to C23, C19 to C24, C20 to C25, C21 to C26, C22 to C27, C23 to C28, C24 to C29, C25 to C30, C26 to C31, C27 to C32, C28 to C33, C29 to C34, C30 to C35, C31 to C36, C32 to C37, C33 to C38, C34 to C39, C35 to C40, C36 to C41, C37 to C42, C38 to C43, C39 to C44, C40 to C45, C41 to C46, J4 to J6, R12 to R14, R13 to R15, R14 to R16, R15 to R17, R16 to R18, R17 to R24, R18 to R25, R19 to R26, R20 to R27, R21 to R28, R22 to R29, SW9 to SW10, SW99 to SW100, SW100 to SW101, SW101 to SW102, SW102 to SW103, SW103 to SW104, SW104 to SW105, SW105 to SW106, SW106 to SW107, SW10 to SW11, SW11 to SW12, SW12 to SW13, SW13 to SW14, SW14 to SW15, SW15 to SW16, SW16 to SW17, SW17 to SW18, SW18 to SW19, SW1 to SW2, SW19 to SW20, SW20 to SW21, SW21 to SW22, SW22 to SW23, SW23 to SW24, SW24 to SW25, SW25 to SW26, SW26 to SW27, SW27 to SW28, SW28 to SW29, SW2 to SW3, SW29 to SW30, SW30 to SW31, SW31 to SW32, SW32 to SW33, SW33 to SW34, SW34 to SW35, SW35 to SW36, SW36 to SW37, SW37 to SW38, SW38 to SW39, SW3 to SW4, SW39 to SW40, SW40 to SW41, SW41 to SW42, SW42 to SW43, SW43 to SW44, SW44 to SW45, SW45 to SW46, SW46 to SW47, SW47 to SW48, SW48 to SW49, SW4 to SW5, SW49 to SW50, SW50 to SW51, SW51 to SW52, SW52 to SW53, SW53 to SW54, SW54 to SW55, SW55 to SW56, SW56 to SW57, SW57 to SW58, SW58 to SW59, SW5 to SW6, SW59 to SW60, SW60 to SW61, SW61 to SW62, SW62 to SW63, SW63 to SW64, SW64 to SW65, SW65 to SW66, SW66 to SW67, SW67 to SW68, SW68 to SW69, SW6 to SW7, SW69 to SW70, SW70 to SW71, SW71 to SW72, SW72 to SW73, SW73 to SW74, SW74 to SW75, SW75 to SW76, SW76 to SW77, SW77 to SW78, SW78 to SW79, SW7 to SW8, SW79 to SW80, SW80 to SW81, SW81 to SW82, SW82 to SW83, SW83 to SW84, SW84 to SW85, SW85 to SW86, SW86 to SW87, SW87 to SW88, SW88 to SW89, SW8 to SW9, SW89 to SW90, SW90 to SW91, SW91 to SW92, SW92 to SW93, SW93 to SW94, SW94 to SW95, SW95 to SW96, SW96 to SW97, SW97 to SW98, SW98 to SW99, U2 to U3, U3 to U4, U4 to U5, U5 to U6, U6 to U7
Connections:
- SW36 pad 2: /FPGA/Kp.NLock -> /Keys/Kp.NLock
- SW37 pad 2: /FPGA/Kp.Slash -> /Keys/Kp.Slash
- SW38 pad 2: /FPGA/Kp.Star -> /Keys/Kp.Star
