File: PCB/clavier.kicad_pcb (KiCad board)
At the start: 4 copper layers, 434 x 134 mm, 209 parts, among them J1 918-418K2023S40001, J2 901-211A1021D10100, J3 901-211A1021D10100, J4 Pin header, 2x4, J5 Pin header, 2x4, J6 TC2050, SW1 DSIC01LS-P, U1 GL852G-OHY60, U2 CH347F, U3 LFE5U-25F-6BG256C, U4 W25Q128JVSIQ, U5 TLV62569DBVR, U6 TLV62569DBVR, U7 TLV62569DBVR, Y1 12MHz, Y1 CO22H4-48.000-WPJDTSTL, Y2 8MHz, Y3 12MHz

Commit message: Improve the CH347F schematics and added 3D models
Parts:
- removed the U4 at (82.7, 79.8)
- removed the Y1 at (142.9, 85.9)
- removed the Y1 at (87.2, 91.9)
- added J7: Pin header, 2x4, Connector_PinHeader_2.54mm:PinHeader_2x04_P2.54mm_Vertical, F.Cu at (463.5, 46.0)
- added J8: Pin header, 2x4, Connector_PinHeader_2.54mm:PinHeader_2x04_P2.54mm_Vertical, F.Cu at (473.7, 70.5)
- added J9: Pin header, 2x4, Connector_PinHeader_2.54mm:PinHeader_2x04_P2.54mm_Vertical, F.Cu at (458.1, 77.3)
- added R30: 1.37kΩ, Resistor_SMD:R_0402_1005Metric_Pad0.72x0.64mm_HandSolder, F.Cu at (452.2, 86.2)
- added R31: 1.65kΩ, Resistor_SMD:R_0402_1005Metric_Pad0.72x0.64mm_HandSolder, F.Cu at (452.2, 88.2)
- added U3: CH347F, Package_DFN_QFN:QFN-28-1EP_4x4mm_P0.4mm_EP2.4x2.4mm, F.Cu at (462.1, 59.1)
- added U8: TLV62569DBVR, Package_TO_SOT_SMD:SOT-23-5, F.Cu at (448.0, 88.9)
- added Y1: 12MHz, Crystal:Crystal_SMD_2520-4Pin_2.5x2.0mm, F.Cu at (482.4, 57.3)
- J1, J2, J3: moved to B.Cu
- J4, J5: footprint Connector_PinHeader_2.54mm:PinHeader_2x04_P2.54mm_Vertical_SMD -> Connector_PinHeader_2.54mm:PinHeader_2x04_P2.54mm_Vertical
- J6: value TC2050 -> Pin header, 2x4; footprint Connector:Tag-Connect_TC2050-IDC-NL_2x05_P1.27mm_Vertical_with_bottom_clip -> Connector_PinHeader_2.54mm:PinHeader_2x04_P2.54mm_Vertical
- R18: value 1kΩ -> 10kΩ
- R19: value 2.55kΩ -> 10kΩ
- R20: value 2.55kΩ -> 1kΩ
- R24: value 11.5kΩ -> 2.55kΩ
- R26: value 4.75kΩ -> 11.5kΩ
- R27: value 1.5kΩ -> 2.55kΩ
- R28: value 1.37kΩ -> 4.75kΩ
- R29: value 1.65kΩ -> 1.5kΩ
- SW10, SW102, SW103, SW104, SW106, SW11, SW12, SW13, SW14, SW15, SW16, SW17, SW18, SW19, SW2, SW20, SW21, SW22, SW23, SW24, SW25, SW26, SW27, SW28, SW29, SW3, SW30, SW31, SW33, SW34, SW35, SW36, SW37, SW38, SW39, SW4, SW41, SW42, SW43, SW44, SW45, SW46, SW47, SW48, SW49, SW5, SW50, SW51, SW52, SW54, SW55, SW56, SW57, SW58, SW59, SW6, SW61, SW62, SW63, SW64, SW65, SW66, SW67, SW68, SW69, SW7, SW70, SW71, SW72, SW73, SW74, SW75, SW78, SW79, SW8, SW80, SW81, SW82, SW83, SW84, SW85, SW86, SW87, SW88, SW9, SW90, SW91, SW92, SW93: footprint Button_Switch_Keyboard:SW_Cherry_MX_1.00u_PCB -> clavier:SW_Cherry_MX_1.00u_PCB
- SW100, SW101, SW77, SW94, SW95, SW96, SW98, SW99: footprint Button_Switch_Keyboard:SW_Cherry_MX_1.25u_PCB -> clavier:SW_Cherry_MX_1.25u_PCB
- SW105, SW32: footprint Button_Switch_Keyboard:SW_Cherry_MX_2.00u_PCB -> clavier:SW_Cherry_MX_2.00u_PCB
- SW107, SW76: footprint Button_Switch_Keyboard:SW_Cherry_MX_2.00u_Vertical_PCB -> clavier:SW_Cherry_MX_2.00u_Vertical_PCB
- SW40: footprint Button_Switch_Keyboard:SW_Cherry_MX_1.50u_PCB -> clavier:SW_Cherry_MX_1.50u_PCB
- SW53: footprint Button_Switch_Keyboard:SW_Cherry_MX_ISOEnter_PCB -> clavier:SW_Cherry_MX_ISOEnter_PCB
- SW60: footprint Button_Switch_Keyboard:SW_Cherry_MX_1.75u_PCB -> clavier:SW_Cherry_MX_1.75u_PCB
- SW89: footprint Button_Switch_Keyboard:SW_Cherry_MX_2.75u_PCB -> clavier:SW_Cherry_MX_2.75u_PCB
- SW97: footprint Button_Switch_Keyboard:SW_Cherry_MX_6.25u_PCB -> clavier:SW_Cherry_MX_6.25u_PCB
- U2: value CH347F -> CH412K; footprint Package_DFN_QFN:QFN-28-1EP_4x4mm_P0.4mm_EP2.4x2.4mm -> Package_TO_SOT_SMD:SOT-363_SC-70-6
- U5: value TLV62569DBVR -> W25Q128JVSIQ; footprint Package_TO_SOT_SMD:SOT-23-5 -> Package_SO:SOIC-8_5.3x5.3mm_P1.27mm
- moved R25 414.6 mm to (477.5, 93.1)
- moved R24 414.3 mm to (477.5, 91.1)
- moved R1 403.5 mm to (472.0, 44.8)
- moved R2 403.5 mm to (472.0, 46.7)
- moved U5 401.5 mm to (461.0, 71.6)
- moved C24 399.7 mm to (486.6, 73.1)
- moved C41 393.0 mm to (446.5, 69.7)
- moved C27 392.3 mm to (467.8, 73.1)
- moved C26 392.3 mm to (467.8, 71.2)
- moved C25 392.3 mm to (467.8, 69.2)
- moved R18 389.2 mm to (464.6, 80.0)
- moved R17 389.2 mm to (464.6, 78.0)
- moved R16 389.2 mm to (464.6, 76.0)
- moved C28 388.9 mm to (482.7, 85.1)
- moved C29 388.9 mm to (482.7, 87.1)
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- renumbered U3 to U4
Connections:
- net Net-(J2-D+) renamed /USB hub/D3+
- net Net-(J2-D-) renamed /USB hub/D3-
- net Net-(J3-D+) renamed /USB hub/D4+
- net Net-(J3-D-) renamed /USB hub/D4-
- C7 pad 2: Net-(U2A-XI) -> Net-(U3A-XI)
- C8 pad 1: Net-(U2A-~{RST}) -> Net-(U3A-~{RST})
- C9 pad 2: Net-(U2A-XO) -> Net-(U3A-XO)
- J4 pad 1: Net-(J4-Pin_1) -> /5-in-1 USB/CH347_SCK
- J4 pad 2: Net-(J4-Pin_2) -> /5-in-1 USB/CH347_MOSI
- J4 pad 3: Net-(J4-Pin_3) -> /5-in-1 USB/CH347_MISO
- J4 pad 4: Net-(J4-Pin_4) -> /5-in-1 USB/CH347_SCS0
- J5 pad 1: Net-(J5-Pin_1) -> /5-in-1 USB/CH347_TCK
- J5 pad 2: Net-(J5-Pin_2) -> /5-in-1 USB/CH347_TDO
- J5 pad 3: Net-(J5-Pin_3) -> /5-in-1 USB/CH347_TDI
- J5 pad 4: Net-(J5-Pin_4) -> /5-in-1 USB/CH347_TMS
- J6 pad 1: +3V3 -> /5-in-1 USB/CH347_TXD0
- J6 pad 2: /FPGA/FPGA config/FPGA_TMS -> /5-in-1 USB/CH347_RXD0
- J6 pad 3: GND -> /5-in-1 USB/CH347_TXD1
- J6 pad 4: /FPGA/FPGA config/FPGA_TCK -> /5-in-1 USB/CH347_RXD1
- J6 pad 5: unconnected-(J6-Pad5) -> GND
- J6 pad 6: /FPGA/FPGA config/FPGA_TDO -> GND
- J6 pad 7: unconnected-(J6-Pad7) -> GND
- J6 pad 8: /FPGA/FPGA config/FPGA_TDI -> GND
- L2 pad 1: Net-(U5-SW) -> Net-(U6-SW)
- L3 pad 1: Net-(U6-SW) -> Net-(U7-SW)
- L4 pad 1: Net-(U7-SW) -> Net-(U8-SW)
- R12 pad 2: Net-(U2A-~{RST}) -> Net-(U3A-~{RST})
- R14 pad 2: /FPGA/FPGA config/Flash_~{CS} -> /5-in-1 USB/CH347_SCL
- R15 pad 2: /FPGA/FPGA config/FPGA_TDO -> /5-in-1 USB/CH347_SDA
- R16 pad 2: /FPGA/FPGA config/FPGA_TDI -> /FPGA/FPGA config/Flash_~{CS}
- R17 pad 2: /FPGA/FPGA config/FPGA_TMS -> /FPGA/FPGA config/FPGA_TDO
- R18 pad 1: /FPGA/FPGA config/FPGA_TCK -> +3V3
- R18 pad 2: GND -> /FPGA/FPGA config/FPGA_TDI
- R19 pad 1: Net-(D2-A) -> +3V3
- R19 pad 2: +3V3 -> /FPGA/FPGA config/FPGA_TMS
- R20 pad 1: Net-(D3-A) -> /FPGA/FPGA config/FPGA_TCK
- R20 pad 2: +3V3 -> GND
- R21 pad 1: Net-(D4-A) -> Net-(D2-A)
- R22 pad 1: Net-(D5-A) -> Net-(D3-A)
- R23 pad 1: Net-(D6-A) -> Net-(D4-A)
- R24 pad 1: +3V3 -> Net-(D5-A)
- R24 pad 2: Net-(U5-FB) -> +3V3
- R25 pad 1: Net-(U5-FB) -> Net-(D6-A)
- R25 pad 2: GND -> +3V3
- R26 pad 1: +2V5 -> +3V3
- R28 pad 1: +1V1 -> +2V5
- SW1 pad 1: Net-(U2A-~{RST}) -> Net-(U3A-~{RST})
- SW36 pad 2: /Keys/Kp.NLock -> /FPGA/Kp.NLock
- SW37 pad 2: /Keys/Kp.Slash -> /FPGA/Kp.Slash
- SW38 pad 2: /Keys/Kp.Star -> /FPGA/Kp.Star
- U1 pad 3: /USB hub/USB_JTAG- -> /5-in-1 USB/USB_JTAG-
- U1 pad 4: /USB hub/USB_JTAG+ -> /5-in-1 USB/USB_JTAG+
- U2 pad 1: Net-(U2A-XI) -> unconnected-(U2-IO1-Pad1)
- U2 pad 2: Net-(U2A-XO) -> GND
- U2 pad 3: Net-(U2A-~{RST}) -> /USB hub/D+
- U2 pad 4: Net-(J5-Pin_1) -> /USB hub/D-
- U2 pad 5: Net-(J5-Pin_2) -> +3V3
- U2 pad 6: +3V3 -> unconnected-(U2-IO4-Pad6)
- U5 pad 1: VBUS -> /FPGA/FPGA config/Flash_~{CS}
- U5 pad 2: GND -> /FPGA/FPGA config/Flash_IO1
- U5 pad 3: Net-(U5-SW) -> /FPGA/FPGA config/Flash_IO2
- U5 pad 4: VBUS -> GND
- U5 pad 5: Net-(U5-FB) -> /FPGA/FPGA config/Flash_IO0
- Y2 pad 1: Net-(U2A-XO) -> Net-(U3A-XO)
- Y2 pad 3: Net-(U2A-XI) -> Net-(U3A-XI)
