File: PCB/display.kicad_sch (KiCad schematic)
At the start: 0 parts

Commit message: Add the USB to JTAG bridge
Parts:
- added D2, D3, D4, D5, D6: LED, LED_SMD:LED_0603_1608Metric_Pad1.05x0.95mm_HandSolder, symbol Device:LED
- added R19, R20, R21, R22, R23: 2.55kΩ, Resistor_SMD:R_0402_1005Metric_Pad0.72x0.64mm_HandSolder, symbol Device:R
Connections:
- new net: D6.2 (A), R23.1
- new net: D2.2 (A), R19.1
- new net: D3.2 (A), R20.1
- new net: D4.2 (A), R21.1
- new net: D5.2 (A), R22.1
- new net +3V3: R19.2, R20.2, R21.2, R22.2, R23.2
- new net LED0: D2.1 (K)
- new net LED1: D3.1 (K)
- new net LED2: D4.1 (K)
- new net LED3: D5.1 (K)
- new net LED4: D6.1 (K)

Commit message: Improve the CH347F schematics and added 3D models
Parts:
- renumbered R19 to R21, R20 to R22, R21 to R23, R22 to R24, R23 to R25
Changed lines of the file:
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@@
 		(on_board yes)
 		(dnp no)
-		(property "Reference" "R23"
+		(property "Reference" "R25"
 			(at 152.4 129.794 90)
 			(effects
@@
 			(project "clavier"
 				(path "/6362c6e0-59ef-40d3-b6e0-7e9dfe7b9b20/7a0fedde-fdbf-441d-b3e6-197cbc93a029"
-					(reference "R23")
+					(reference "R25")
 					(unit 1)
 				)
@@
 		(on_board yes)
 		(dnp no)
-		(property "Reference" "R20"
+		(property "Reference" "R22"
 			(at 152.4 91.694 90)
 			(effects
@@
 			(project "clavier"
 				(path "/6362c6e0-59ef-40d3-b6e0-7e9dfe7b9b20/7a0fedde-fdbf-441d-b3e6-197cbc93a029"
-					(reference "R20")
+					(reference "R22")
 					(unit 1)
 				)
@@
 		(dnp no)
 		(fields_autoplaced yes)
-		(property "Reference" "#PWR065"
+		(property "Reference" "#PWR069"
 			(at 165.1 67.31 0)
 			(effects
@@
 			(project "clavier"
 				(path "/6362c6e0-59ef-40d3-b6e0-7e9dfe7b9b20/7a0fedde-fdbf-441d-b3e6-197cbc93a029"
-					(reference "#PWR065")
+					(reference "#PWR069")
 					(unit 1)
 				)
@@
 		(on_board yes)
 		(dnp no)
-		(property "Reference" "R21"
+		(property "Reference" "R23"
 			(at 152.4 104.394 90)
 			(effects
@@
 			(project "clavier"
 				(path "/6362c6e0-59ef-40d3-b6e0-7e9dfe7b9b20/7a0fedde-fdbf-441d-b3e6-197cbc93a029"
-					(reference "R21")
+					(reference "R23")
 					(unit 1)
 				)
@@
 		(on_board yes)
 		(dnp no)
-		(property "Reference" "R19"
+		(property "Reference" "R21"
 			(at 152.4 78.994 90)
 			(effects
@@
 			(project "clavier"
 				(path "/6362c6e0-59ef-40d3-b6e0-7e9dfe7b9b20/7a0fedde-fdbf-441d-b3e6-197cbc93a029"
-					(reference "R19")
+					(reference "R21")
 					(unit 1)
 				)
@@
 		(on_board yes)
 		(dnp no)
-		(property "Reference" "R22"
+		(property "Reference" "R24"
 			(at 152.4 117.094 90)
 			(effects
@@
 			(project "clavier"
 				(path "/6362c6e0-59ef-40d3-b6e0-7e9dfe7b9b20/7a0fedde-fdbf-441d-b3e6-197cbc93a029"
-					(reference "R22")
-					(unit 1)
-				)
+					(reference "R24")
+					(unit 1)
+				)

Commit message: Add LICENSE and minor improvements
- Filled the title blocks
- Connected the LEDs to the FPGA
- Changed the FPGA programming header
- Added USB fuse and capacitors
Other:
- company: (none) -> Copyright (c) 2025 L. Sartory
- title: (none) -> Clavier - Display
Changed lines of the file:
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@@
 	(generator_version "9.0")
 	(paper "A4")
+	(title_block
+		(title "Clavier - Display")
+		(date "2025-06-01")
+		(rev "1.0")
+		(company "Copyright (c) 2025 L. Sartory")
+		(comment 1 "SPDX-License-Identifier: CERN-OHL-P-2.0")
+	)
 	(junction
 		(at 165.1 114.3)
@@
 		(dnp no)
 		(fields_autoplaced yes)
-		(property "Reference" "#PWR069"
+		(property "Reference" "#PWR068"
 			(at 165.1 67.31 0)
 			(effects
@@
 			(project "clavier"
 				(path "/6362c6e0-59ef-40d3-b6e0-7e9dfe7b9b20/7a0fedde-fdbf-441d-b3e6-197cbc93a029"
-					(reference "#PWR069")
+					(reference "#PWR068")
 					(unit 1)
 				)

Commit message: Add the first row of keycaps
Parts:
- renumbered R21 to R27, R22 to R28, R23 to R29, R24 to R30, R25 to R31
Changed lines of the file:
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@@
 		(on_board yes)
 		(dnp no)
-		(property "Reference" "R25"
+		(property "Reference" "R31"
 			(at 152.4 129.794 90)
 			(effects
@@
 			(project "clavier"
 				(path "/6362c6e0-59ef-40d3-b6e0-7e9dfe7b9b20/7a0fedde-fdbf-441d-b3e6-197cbc93a029"
-					(reference "R25")
+					(reference "R31")
 					(unit 1)
 				)
@@
 		(on_board yes)
 		(dnp no)
-		(property "Reference" "R22"
+		(property "Reference" "R28"
 			(at 152.4 91.694 90)
 			(effects
@@
 			(project "clavier"
 				(path "/6362c6e0-59ef-40d3-b6e0-7e9dfe7b9b20/7a0fedde-fdbf-441d-b3e6-197cbc93a029"
-					(reference "R22")
+					(reference "R28")
 					(unit 1)
 				)
@@
 		(dnp no)
 		(fields_autoplaced yes)
-		(property "Reference" "#PWR068"
+		(property "Reference" "#PWR077"
 			(at 165.1 67.31 0)
 			(effects
@@
 			(project "clavier"
 				(path "/6362c6e0-59ef-40d3-b6e0-7e9dfe7b9b20/7a0fedde-fdbf-441d-b3e6-197cbc93a029"
-					(reference "#PWR068")
+					(reference "#PWR077")
 					(unit 1)
 				)
@@
 		(on_board yes)
 		(dnp no)
-		(property "Reference" "R23"
+		(property "Reference" "R29"
 			(at 152.4 104.394 90)
 			(effects
@@
 			(project "clavier"
 				(path "/6362c6e0-59ef-40d3-b6e0-7e9dfe7b9b20/7a0fedde-fdbf-441d-b3e6-197cbc93a029"
-					(reference "R23")
+					(reference "R29")
 					(unit 1)
 				)
@@
 		(on_board yes)
 		(dnp no)
-		(property "Reference" "R21"
+		(property "Reference" "R27"
 			(at 152.4 78.994 90)
 			(effects
@@
 			(project "clavier"
 				(path "/6362c6e0-59ef-40d3-b6e0-7e9dfe7b9b20/7a0fedde-fdbf-441d-b3e6-197cbc93a029"
-					(reference "R21")
+					(reference "R27")
 					(unit 1)
 				)
@@
 		(on_board yes)
 		(dnp no)
-		(property "Reference" "R24"
+		(property "Reference" "R30"
 			(at 152.4 117.094 90)
 			(effects
@@
 			(project "clavier"
 				(path "/6362c6e0-59ef-40d3-b6e0-7e9dfe7b9b20/7a0fedde-fdbf-441d-b3e6-197cbc93a029"
-					(reference "R24")
-					(unit 1)
-				)
+					(reference "R30")
+					(unit 1)
+				)

Commit message: Place and route peripheral components
Parts:
- renumbered R27 to R28, R28 to R29, R29 to R30, R30 to R31, R31 to R32
Changed lines of the file:
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@@
 		(on_board yes)
 		(dnp no)
-		(property "Reference" "R31"
+		(property "Reference" "R32"
 			(at 152.4 129.794 90)
 			(effects
@@
 			(project "clavier"
 				(path "/6362c6e0-59ef-40d3-b6e0-7e9dfe7b9b20/7a0fedde-fdbf-441d-b3e6-197cbc93a029"
-					(reference "R31")
+					(reference "R32")
 					(unit 1)
 				)
@@
 		(on_board yes)
 		(dnp no)
-		(property "Reference" "R28"
+		(property "Reference" "R29"
 			(at 152.4 91.694 90)
 			(effects
@@
 			(project "clavier"
 				(path "/6362c6e0-59ef-40d3-b6e0-7e9dfe7b9b20/7a0fedde-fdbf-441d-b3e6-197cbc93a029"
-					(reference "R28")
+					(reference "R29")
 					(unit 1)
 				)
@@
 		(on_board yes)
 		(dnp no)
-		(property "Reference" "R29"
+		(property "Reference" "R30"
 			(at 152.4 104.394 90)
 			(effects
@@
 			(project "clavier"
 				(path "/6362c6e0-59ef-40d3-b6e0-7e9dfe7b9b20/7a0fedde-fdbf-441d-b3e6-197cbc93a029"
-					(reference "R29")
+					(reference "R30")
 					(unit 1)
 				)
@@
 		(on_board yes)
 		(dnp no)
-		(property "Reference" "R27"
+		(property "Reference" "R28"
 			(at 152.4 78.994 90)
 			(effects
@@
 			(project "clavier"
 				(path "/6362c6e0-59ef-40d3-b6e0-7e9dfe7b9b20/7a0fedde-fdbf-441d-b3e6-197cbc93a029"
-					(reference "R27")
+					(reference "R28")
 					(unit 1)
 				)
@@
 		(on_board yes)
 		(dnp no)
-		(property "Reference" "R30"
+		(property "Reference" "R31"
 			(at 152.4 117.094 90)
 			(effects
@@
 			(project "clavier"
 				(path "/6362c6e0-59ef-40d3-b6e0-7e9dfe7b9b20/7a0fedde-fdbf-441d-b3e6-197cbc93a029"
-					(reference "R30")
-					(unit 1)
-				)
+					(reference "R31")
+					(unit 1)
+				)
