File: PCB/keys.kicad_sch (KiCad schematic)
At the start: 106 parts

Commit message: Complete the PCB routing
Parts:
- renumbered SW2 to SW1, SW11 to SW10, SW99 to SW100, SW100 to SW101, SW101 to SW102, SW102 to SW103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
