File: PCB/usb_hub.kicad_sch (KiCad schematic)
At the start: 30 parts, among them J10 901-211A1021D10100, J7 918-418K2023S40001, J9 901-211A1021D10100, U16 GL852G-OHY60, Y2 12MHz

Commit message: Fix DRC errors and warnings
Parts:
- J10, J9: footprint Connector_USB:USB_A_Molex_67643_Horizontal -> clavier:USB_A_Molex_67643_Horizontal
Changed lines of the file:
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@@
 			)
 		)
-		(property "Footprint" "Connector_USB:USB_A_Molex_67643_Horizontal"
+		(property "Footprint" "clavier:USB_A_Molex_67643_Horizontal"
 			(at 232.41 97.79 0)
 			(effects
@@
 			)
 		)
-		(property "Footprint" "Connector_USB:USB_A_Molex_67643_Horizontal"
+		(property "Footprint" "clavier:USB_A_Molex_67643_Horizontal"
 			(at 232.41 142.24 0)
 			(effects
